File: PCB/Breakouts/breakout.kicad_pcb (KiCad board)
At the start: 2 copper layers, 100 x 95 mm, 14 parts, among them J1 Conn_01x06_Male, J4 Hall, U1 Joystick_XY, U2 Joystick_Z

Commit message: Breakouts V-Cut update, Zipped Gerbers
Parts:
- J1: value Conn_01x06_Male -> (none)
Other:
- board size 100 x 95 mm -> 100 x 100 mm
Changed lines of the file:
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@@
   (general
     (thickness 1.6)
-    (drawings 15)
+    (drawings 42)
     (tracks 51)
     (zones 0)
@@
       (plotinvisibletext false)
       (padsonsilk false)
-      (subtractmaskfromsilk false)
+      (subtractmaskfromsilk true)
       (outputformat 1)
       (mirror false)
@@
       (effects (font (size 1 1) (thickness 0.15)))
     )
-    (fp_text value Conn_01x06_Male (at 0 15.03 90) (layer F.Fab)
+    (fp_text value "" (at 0 16.62 90) (layer F.Fab)
       (effects (font (size 1 1) (thickness 0.15)))
     )
@@
     (pad 1 np_thru_hole circle (at 0 0) (size 3.2 3.2) (drill 3.2) (layers *.Cu *.Mask))
   )
-  (gr_line (start 120 105) (end 145 105) (layer Edge.Cuts) (width 0.15))
-  (gr_text "Hall Sensor" (at 133 115) (layer F.SilkS)
+  (gr_circle (center 119 108) (end 119.25 108) (layer Edge.Cuts) (width 0.15))
+  (gr_circle (center 119 106) (end 119.25 106) (layer Edge.Cuts) (width 0.15))
+  (gr_circle (center 119 109) (end 119.25 109) (layer Edge.Cuts) (width 0.15))
+  (gr_circle (center 119 107) (end 119.25 107) (layer Edge.Cuts) (width 0.15))
+  (gr_line (start 143 110) (end 143 130) (layer Edge.Cuts) (width 0.15))
+  (gr_line (start 145 110) (end 145 130) (layer Edge.Cuts) (width 0.15))
+  (gr_line (start 145 130) (end 145 135) (layer Edge.Cuts) (width 0.15))
+  (gr_circle (center 144 133) (end 144.25 133) (layer Edge.Cuts) (width 0.15))
+  (gr_circle (center 144 108) (end 144.25 108) (layer Edge.Cuts) (width 0.15))
+  (gr_circle (center 144 106) (end 144.25 106) (layer Edge.Cuts) (width 0.15))
+  (gr_circle (center 144 109) (end 144.25 109) (layer Edge.Cuts) (width 0.15))
+  (gr_circle (center 144 107) (end 144.25 107) (layer Edge.Cuts) (width 0.15))
+  (gr_line (start 145 110) (end 143 110) (layer Edge.Cuts) (width 0.15))
+  (gr_line (start 145 110) (end 145 105) (layer Edge.Cuts) (width 0.15))
+  (gr_circle (center 144 131) (end 144.25 131) (layer Edge.Cuts) (width 0.15))
+  (gr_line (start 143 130) (end 145 130) (layer Edge.Cuts) (width 0.15))
+  (gr_line (start 143 130) (end 143 135) (layer Edge.Cuts) (width 0.15))
+  (gr_line (start 143 110) (end 143 105) (layer Edge.Cuts) (width 0.15))
+  (gr_circle (center 144 132) (end 144.25 132) (layer Edge.Cuts) (width 0.15))
+  (gr_circle (center 144 134) (end 144.25 134) (layer Edge.Cuts) (width 0.15))
+  (gr_line (start 120 130) (end 120 135) (layer Edge.Cuts) (width 0.15))
+  (gr_line (start 120 110) (end 120 130) (layer Edge.Cuts) (width 0.15))
+  (gr_line (start 118 110) (end 118 130) (layer Edge.Cuts) (width 0.15))
+  (gr_line (start 118 130) (end 118 135) (layer Edge.Cuts) (width 0.15))
+  (gr_line (start 118 110) (end 118 105) (layer Edge.Cuts) (width 0.15))
+  (gr_line (start 120 110) (end 120 105) (layer Edge.Cuts) (width 0.15))
+  (gr_circle (center 119 132) (end 119.25 132) (layer Edge.Cuts) (width 0.15))
+  (gr_circle (center 119 131) (end 119.25 131) (layer Edge.Cuts) (width 0.15))
+  (gr_circle (center 119 134) (end 119.25 134) (layer Edge.Cuts) (width 0.15))
+  (gr_circle (center 119 133) (end 119.25 133) (layer Edge.Cuts) (width 0.15))
+  (gr_line (start 120 110) (end 118 110) (layer Edge.Cuts) (width 0.15))
+  (gr_line (start 118 130) (end 120 130) (layer Edge.Cuts) (width 0.15))
+  (gr_line (start 95 105) (end 195 105) (layer Edge.Cuts) (width 0.15))
+  (gr_line (start 195 135) (end 195 105) (layer Edge.Cuts) (width 0.15))
+  (gr_line (start 95 135) (end 195 135) (layer Edge.Cuts) (width 0.15))
+  (gr_line (start 95 105) (end 95 135) (layer Edge.Cuts) (width 0.15))
+  (gr_text "Hall Sensor" (at 131.5 131.25) (layer F.SilkS)
     (effects (font (size 1.5 1.5) (thickness 0.3)))
   )
-  (gr_line (start 120 130) (end 120 105) (layer Edge.Cuts) (width 0.15))
-  (gr_line (start 145 105) (end 145 130) (layer Edge.Cuts) (width 0.15))
-  (gr_line (start 145 130) (end 120 130) (layer Edge.Cuts) (width 0.15))
   (gr_text "Joystick Controller" (at 146 99) (layer F.SilkS)
     (effects (font (size 1.5 1.5) (thickness 0.3)))
   )
-  (gr_text "Hall Sensor" (at 108 115) (layer F.SilkS)
+  (gr_text "Hall Sensor" (at 106 131) (layer F.SilkS)
     (effects (font (size 1.5 1.5) (thickness 0.3)))
   )
-  (gr_line (start 95 130) (end 95 105) (layer Edge.Cuts) (width 0.15))
-  (gr_line (start 120 130) (end 95 130) (layer Edge.Cuts) (width 0.15))
-  (gr_line (start 120 105) (end 120 130) (layer Edge.Cuts) (width 0.15))
-  (gr_line (start 95 105) (end 120 105) (layer Edge.Cuts) (width 0.15))
   (gr_line (start 195 35) (end 95 35) (layer Edge.Cuts) (width 0.15))
   (gr_line (start 195 105) (end 195 35) (layer Edge.Cuts) (width 0.15))
-  (gr_line (start 95 105) (end 195 105) (layer Edge.Cuts) (width 0.15))
   (gr_line (start 95 35) (end 95 105) (layer Edge.Cuts) (width 0.15))
   (segment (start 125 120) (end 133 120) (width 0.25) (layer B.Cu) (net 0))
@@
   (segment (start 100 122.54) (end 108 122.54) (width 0.25) (layer B.Cu) (net 11))
   (segment (start 100 125.08) (end 108 125.08) (width 0.25) (layer B.Cu) (net 12))
+  (zone (net 1) (net_name "Net-(D1-Pad1)") (layer F.Cu) (hatch edge 0.508)
+    (connect_pads (clearance 0.508))
+    (min_thickness 0.254)
+    (fill yes (arc_segments 16) (thermal_gap 0.508) (thermal_bridge_width 0.508))
+    (polygon
+      (pts
+        (xy 95 35) (xy 195 35) (xy 195 105) (xy 95 105)
+      )
+    )
+  )
   (zone (net 1) (net_name "Net-(D1-Pad1)") (layer B.Cu) (hatch edge 0.508)
     (connect_pads (clearance 0.508))
@@
     )
   )
-  (zone (net 1) (net_name "Net-(D1-Pad1)") (layer F.Cu) (hatch edge 0.508)
+  (zone (net 11) (net_name "Net-(J2-Pad2)") (layer F.Cu) (hatch edge 0.508)
     (connect_pads (clearance 0.508))
     (min_thickness 0.254)
@@
     (polygon
       (pts
-        (xy 95 35) (xy 195 35) (xy 195 105) (xy 95 105)
+        (xy 95 105) (xy 118 105) (xy 118 135) (xy 95 135)
+      )
+    )
+  )
+  (zone (net 0) (net_name "") (layer F.Cu) (hatch edge 0.508)
+    (connect_pads (clearance 0.508))
+    (min_thickness 0.254)
+    (fill yes (arc_segments 16) (thermal_gap 0.508) (thermal_bridge_width 0.508))
+    (polygon
+      (pts
+        (xy 120 105) (xy 143 105) (xy 143 135) (xy 120 135)
       )
     )
@@
     (polygon
       (pts
-        (xy 95 105) (xy 120 105) (xy 120 130) (xy 95 130)
-      )
-    )
-  )
-  (zone (net 11) (net_name "Net-(J2-Pad2)") (layer F.Cu) (hatch edge 0.508)
-    (connect_pads (clearance 0.508))
-    (min_thickness 0.254)
-    (fill yes (arc_segments 16) (thermal_gap 0.508) (thermal_bridge_width 0.508))
-    (polygon
-      (pts
-        (xy 95 105) (xy 95 130) (xy 120 130) (xy 120 105)
+        (xy 95 105) (xy 118 105) (xy 118 135) (xy 95 135)
       )
     )
@@
     (polygon
       (pts
-        (xy 120 105) (xy 145 105) (xy 145 130) (xy 120 130)
+        (xy 120 105) (xy 143 105) (xy 143 135) (xy 120 135)
       )
     )
-  )
-  (zone (net 0) (net_name "") (layer F.Cu) (hatch edge 0.508)
-    (connect_pads (clearance 0.508))
-    (min_thickness 0.254)
-    (fill yes (arc_segments 16) (thermal_gap 0.508) (thermal_bridge_width 0.508))
-    (polygon
-      (pts
-        (xy 120 105) (xy 120 130) (xy 145 130) (xy 145 105)
-      )
-    )
